File: PCB v0.1.kicad_pcb (KiCad board)
At the start: 2 copper layers, 100 x 100 mm, 61 parts, among them J1 XT60 M (Vertical), J10 2.54mm 3P, J11 2.54mm 3P, J12 2.54mm 3P, J13 JST-SH 3P, J14 JST-SH 3P, J15 JST-SH 3P, J16 JST-SH 3P, J17 JST-SH 3P, J18 JST-SH 3P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

Commit message: Rev A finished. docs made, BOM made.
Parts:
- J1: value XT60 M (Vertical) -> XT60 M (Horizontal)
- J4, J5, J6, J7, J8: value Screw Terminal 5P -> Screw 2.54mm 5P
- moved J18 89.5 mm to (150.5, 44.2), turned to 0 degrees
- moved J13 86.4 mm to (191.3, 44.2), turned to 0 degrees
- moved J17 83.2 mm to (158.7, 44.2), turned to 0 degrees
- moved J14 81.2 mm to (183.1, 44.2), turned to 0 degrees
- moved J16 79.6 mm to (166.8, 44.2), turned to 0 degrees
- moved J15 78.9 mm to (175.0, 44.2), turned to 0 degrees
- moved J6 29.5 mm to (105.7, 74.4)
- moved J8 27.0 mm to (133.6, 74.4)
- moved J3 10.3 mm to (116.1, 51.3), turned to -90 degrees
- moved J4 10.3 mm to (130.0, 51.3), turned to -90 degrees
- moved J5 10.3 mm to (144.0, 51.3), turned to -90 degrees
- moved H2 4.44 mm to (106.9, 137.2)
- moved C3 4.26 mm to (187.5, 75.7)
- moved C4 4.26 mm to (179.8, 75.7)
- moved C6 4.26 mm to (178.3, 84.7)
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Connections:
- A1 pad 10: /REV_2 -> /ENC_5
- A1 pad 14: /BLDC_4 -> /BLDC_0
- A1 pad 15: /REV_4 -> /REV_0
- A1 pad 16: /BLDC_5 -> /BLDC_1
- A1 pad 17: /REV_5 -> /REV_1
- A1 pad 19: /SERVO_0 -> /BLDC_2
- A1 pad 20: /SERVO_1 -> /REV_2
- A1 pad 21: /ENC_0 -> /SERVO_0
- A1 pad 22: /ENC_1 -> /SERVO_1
- A1 pad 24: /ENC_2 -> /SERVO_2
- A1 pad 25: /ENC_3 -> /SERVO_3
- A1 pad 26: /ENC_4 -> /BLDC_5
- A1 pad 27: /ENC_5 -> /REV_5
- A1 pad 32: /SERVO_2 -> /BLDC_4
- A1 pad 34: /SERVO_3 -> /REV_4
- A1 pad 4: /BLDC_0 -> /ENC_0
- A1 pad 5: /REV_0 -> /ENC_1
- A1 pad 6: /BLDC_1 -> /ENC_2
- A1 pad 7: /REV_1 -> /ENC_3
- A1 pad 9: /BLDC_2 -> /ENC_4
Routing:
- net /ENC_0: track 58.1 -> 5.86 mm
- net /ENC_5: track 77.2 -> 28.2 mm
- net /ENC_4: track 70.2 -> 22.5 mm
- net /ENC_1: track 52.5 -> 8.26 mm
- net /ENC_3: track 63.1 -> 19.5 mm
- net +5.1V: track 109.6 -> 152.8 mm
- net /ENC_2: track 55.6 -> 13.9 mm
- net /BLDC_5: track 66.1 -> 29.2 mm
- net /REV_0: track 90.2 -> 55.1 mm
- net /REV_2: track 46.7 -> 11.9 mm
- net /REV_1: track 69.6 -> 35.8 mm
- net /REV_5: track 66.7 -> 34.9 mm
- net /SERVO_1: track 91.4 -> 61.3 mm, vias 1 -> 0
- net /BLDC_1: track 69.3 -> 40.5 mm
- net /BLDC_0: track 89.2 -> 60.8 mm
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Other:
- board text added: "Designed by: Ilo Japar"
- board text added: "HKU ROVER TEAM"
- board text added: "POWER"
- board text added: "Prototype Rover PCB v0.1 rev A"
- board text added: "SERVOS"
- board text removed: "POW"

Commit message: Created new layout, fixed XT30 polarity
Parts:
- J1: value XT60 M (Horizontal) -> XT60 M (Vertical)
- J4, J5, J6, J7, J8: value Screw 2.54mm 5P -> Screw Terminal 5P
- U1, U2: value AMASS_XT30PW-M_1x02_P2.50mm_Horizontal -> AMASS_XT30PW-F_1x02_P2.50mm_Horizontal; footprint Connector_AMASS:AMASS_XT30PW-M_1x02_P2.50mm_Horizontal -> Connector_AMASS:AMASS_XT30PW-F_1x02_P2.50mm_Horizontal
- U3: moved to B.Cu
- moved R6 91.6 mm to (84.6, 52.8)
- moved R7 91.6 mm to (88.4, 52.8)
- moved R4 91.6 mm to (80.8, 52.8)
- moved R5 91.6 mm to (77.2, 52.8)
- moved R8 91.6 mm to (92.2, 52.8)
- moved D5 67.7 mm to (171.2, 62.5), turned to -90 degrees
- moved D6 67.3 mm to (175.4, 62.5), turned to -90 degrees
- moved D7 66.9 mm to (179.7, 62.5), turned to -90 degrees
- moved D8 66.5 mm to (183.9, 62.5), turned to -90 degrees
- moved J6 57.4 mm to (156.0, 46.7)
- moved J7 57.2 mm to (169.7, 46.7)
- moved J8 57.0 mm to (183.4, 46.7)
- moved A1 53.4 mm to (177.3, 114.3), turned to 0 degrees
- moved C8 51.0 mm to (154.7, 84.4), turned to -90 degrees
- moved J18 49.3 mm to (189.2, 74.7)
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Connections:
- A1 pad 10: /ENC_5 -> /REV_3
- A1 pad 11: /BLDC_3 -> /BLDC_2
- A1 pad 12: /REV_3 -> /REV_2
- A1 pad 14: /BLDC_0 -> /BLDC_1
- A1 pad 15: /REV_0 -> /REV_1
- A1 pad 16: /BLDC_1 -> /SERVO_0
- A1 pad 17: /REV_1 -> /SERVO_1
- A1 pad 19: /BLDC_2 -> /SERVO_2
- A1 pad 20: /REV_2 -> /SERVO_3
- A1 pad 21: /SERVO_0 -> /REV_5
- A1 pad 22: /SERVO_1 -> /BLDC_5
- A1 pad 24: /SERVO_2 -> /ENC_2
- A1 pad 25: /SERVO_3 -> /ENC_1
- A1 pad 26: /BLDC_5 -> /ENC_0
- A1 pad 27: /REV_5 -> /ENC_3
- A1 pad 32: /BLDC_4 -> /ENC_4
- A1 pad 34: /REV_4 -> /ENC_5
- A1 pad 4: /ENC_0 -> /REV_4
- A1 pad 5: /ENC_1 -> /BLDC_4
- A1 pad 6: /ENC_2 -> /REV_0
- A1 pad 7: /ENC_3 -> /BLDC_0
- A1 pad 9: /ENC_4 -> /BLDC_3
Routing:
- net /ENC_0: track 5.86 -> 79.9 mm
- net /BLDC_5: track 29.2 -> 102.3 mm, vias 0 -> 1
- net /PICO_INT: track 85.8 -> 13.5 mm, vias 1 -> 0
- net /REV_2: track 11.9 -> 83.2 mm, vias 0 -> 1
- net /REV_5: track 34.9 -> 103.5 mm, vias 0 -> 1
- net +5.1V: track 152.8 -> 85.1 mm, vias 8 -> 1
- net /REV_1: track 35.8 -> 102.0 mm, vias 0 -> 1
- net /PICO_EN: track 79.2 -> 16.1 mm, vias 1 -> 0
- net /ENC_1: track 8.26 -> 70.6 mm
- net /BLDC_2: track 17.6 -> 79.6 mm, vias 0 -> 1
- net /BLDC_1: track 40.5 -> 97.6 mm, vias 0 -> 1
- net +12V: track 55.1 -> 0.00 mm, vias 98 -> 0
- net /ENC_3: track 19.5 -> 71.6 mm
- net /ENC_2: track 13.9 -> 64.3 mm
- net /SERVO_3: track 67.7 -> 22.6 mm
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- added copper zone on B.Cu, net Net-(FB1-Pad1)
- removed copper zone on B.Cu, net +12V
- removed copper zone on B.Cu, net +BATT
- removed copper zone on B.Cu, net GND
- removed copper zone on F.Cu, net GND
Other:
- board size 100 x 100 mm -> 77.4 x 97 mm

Commit message: v0.2. Corrected XT30 polarity, less than 10x10cm in size
Parts:
- removed U3: 3.2~32V -> 5.1V 5A, Library:Buck_Converter_44x22mm
- J1: value XT60 M (Vertical) -> XT60 M (Horizontal)
- moved R5 80.8 mm to (157.9, 54.9), turned to 90 degrees
- moved R4 79.5 mm to (160.2, 54.9), turned to -90 degrees
- moved R6 78.0 mm to (162.5, 54.9), turned to -90 degrees
- moved R7 76.4 mm to (164.8, 54.9), turned to -90 degrees
- moved R8 74.9 mm to (167.1, 54.9), turned to -90 degrees
- moved FB2 15.3 mm to (177.8, 95.8)
- moved F3 15.1 mm to (177.8, 93.2), turned to 0 degrees
- moved C10 15.1 mm to (139.7, 108.6)
- moved C11 15.1 mm to (139.7, 120.1)
- moved C8 15.1 mm to (139.7, 85.3)
- moved C9 15.1 mm to (139.7, 96.9)
- moved J13 15.0 mm to (150.8, 55.6)
- moved J16 15.0 mm to (174.2, 55.6)
- moved J1 15.0 mm to (122.9, 126.5)
- moved J5 15.0 mm to (127.2, 47.2)
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Connections:
- J1 pad : (no net) -> GND
- U1 pad : (no net) -> GND (x2)
- U2 pad : (no net) -> GND (x2)
Routing:
- net +BATT: track 44.9 -> 165.7 mm
- net +7.5V: track 0.00 -> 99.9 mm, vias 0 -> 3
- net GND: track 0.00 -> 25.5 mm, vias 0 -> 331
- net +12V: track 0.00 -> 25.3 mm, vias 0 -> 1
- net +5.1V: track 85.1 -> 101.1 mm
- net Net-(D5-K): track 0.00 -> 8.36 mm, vias 0 -> 2
- net Net-(D6-K): track 0.00 -> 7.55 mm
- net Net-(D8-K): track 0.00 -> 7.35 mm
- net Net-(D7-K): track 0.00 -> 6.74 mm
- net Net-(R4-Pad1): track 0.00 -> 2.51 mm
- net /ENC_4: track 49.4 -> 51.5 mm
- net /ENC_3: track 71.6 -> 73.6 mm
- net /ENC_0: track 79.9 -> 81.7 mm
- net /ENC_1: track 70.6 -> 72.4 mm
- net /ENC_2: track 64.3 -> 65.9 mm
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- added copper zone on B.Cu, net GND
- added copper zone on F.Cu, net GND
Other:
- board text added: "12V IN →"
- board text added: "7.5V IN →"
- board text added: "BATTERY IN →"
- board text added: "ENCODERS"
- board text added: "HKU MARTIANS"
- board text added: "J3-8"
- board text added: "Prototype Rover PCB v0.2 rev A"
- board text removed: "DC MOTOR ENCODERS"
- board text removed: "HKU ROVER TEAM"
- board text removed: "Prototype Rover PCB v0.1 rev A"
