File: PCB v0.2.kicad_sch (KiCad schematic)
At the start: 61 parts, among them J1 XT60-M, J10 Screw 2.54mm 5P, J11 Screw 2.54mm 5P, J12 Screw 2.54mm 5P, J13 2.54mm 3P, J14 2.54mm 3P, J15 2.54mm 3P, J16 2.54mm 3P, J17 JST-SH 3P, J18 JST-SH 3P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

Commit message: U1 symbol was not in v0.2
Parts:
- added TP1, TP2, TP3, TP4, TP5, TP6: TestPoint, TestPoint:TestPoint_Pad_D1.5mm, symbol Connector:TestPoint
- J10, J11, J12, J7, J8, J9: footprint Connector_PinHeader_2.54mm:PinHeader_1x05_P2.54mm_Vertical -> TerminalBlock:TerminalBlock_Xinya_XY308-2.54-5P_1x05_P2.54mm_Horizontal
- U1: footprint Library:Buck_Converter_44x22mm -> Library:Buck_Converter_54x24mm
Connections:
- net +12V: now also TP3.1
- net +3V3: now also TP2.1
- net +5.1V: now also TP6.1
- net +7.5V: now also TP4.1
- net +BATT: now also TP1.1
- net ADC_IN: now also TP5.1
Other:
- moved on the sheet: J3, J4, J5, J6
